File: main.kicad_sch (KiCad schematic)
At the start: 35 parts, among them J1 inductor connector, J2 inductor connector, J3 test point, J4 test point, J5 IN, J6 pulse width selector, Q1 T60NO2R, U1 NE555P, U2 NE555P

Commit message: more details
Parts:
- added F1: 2A, Resistor_SMD:R_MELF_MMB-0207, symbol Device:Polyfuse
- D1: value 1N4148 -> SS34
Connections:
- net VCC: now also F1.1; no longer D2.2 (A)
- new net: D2.2 (A), F1.2
Other:
- note added: ">60A surge current rating"
- moved on the sheet: C1, C10, C11, C12, C13, C14, C2, C3, C4, C5, C6, C7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

Commit message: Changed gate resistor Add heat map
Parts:
- R5: value 62 -> 10k
Connections:
- net GATE: now also R5.1, U1.3 (Q); no longer Q1.1 (G), R5.2
- new net: Q1.1 (G), R5.2
Other:
- note added: "Min value 62 Ohm to protect 555 Low value (~100) drives MOSFET harder but causes gate "ringing" on turn-on High value (~10k) dampens ringing but causes switching loss and heat"
- moved on the sheet: R5
Changed lines of the file:
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@@
+    (stroke (width 0) (type default) (color 0 0 0 0))
+  )
+  (wire (pts (xy 198.12 101.6) (xy 203.835 101.6))
     (stroke (width 0) (type default) (color 0 0 0 0))
   )
@@
     (stroke (width 0) (type default) (color 0 0 0 0))
   )
-  (wire (pts (xy 200.025 101.6) (xy 203.835 101.6))
+  (wire (pts (xy 186.055 101.6) (xy 190.5 101.6))
     (stroke (width 0) (type default) (color 0 0 0 0))
   )
@@
     (stroke (width 0) (type default) (color 0 0 0 0))
   )
-  (wire (pts (xy 138.43 89.535) (xy 136.525 89.535))
-    (stroke (width 0) (type default) (color 0 0 0 0))
-  )
   (wire (pts (xy 219.71 48.26) (xy 231.14 48.26))
     (stroke (width 0) (type default) (color 0 0 0 0))
   )
-  (wire (pts (xy 149.225 89.535) (xy 146.05 89.535))
+  (wire (pts (xy 136.525 89.535) (xy 141.605 89.535))
     (stroke (width 0) (type default) (color 0 0 0 0))
   )
@@
     (effects (font (size 1.27 1.27)) (justify left bottom))
   )
-  (text "Low Rds(on)\nLow Cgate" (at 191.77 109.855 0)
+  (text "Low Rds(on)\nLow Cgate" (at 224.79 103.505 0)
     (effects (font (size 1.27 1.27)) (justify left bottom))
   )
@@
     (effects (font (size 1.27 1.27)) (justify left bottom))
   )
-  (text "Monostable oscilator\nwith variable pulse width" (at 153.035 99.695 0)
+  (text "Monostable oscilator\nwith variable pulse width" (at 150.495 99.695 0)
     (effects (font (size 1.27 1.27)) (justify left bottom))
   )
   (text "~50Hz trigger" (at 86.36 92.075 0)
+    (effects (font (size 1.27 1.27)) (justify left bottom))
+  )
+  (text "Min value 62 Ohm to protect 555\nLow value (~100) drives MOSFET harder \nbut causes gate \"ringing\" on turn-on \nHigh value (~10k) dampens ringing\nbut causes switching loss and heat\n"
+    (at 171.45 115.57 0)
     (effects (font (size 1.27 1.27)) (justify left bottom))
   )
@@
     )
   )
-  (global_label "GATE" (shape input) (at 149.225 89.535 0) (fields_autoplaced)
+  (global_label "GATE" (shape input) (at 141.605 89.535 0) (fields_autoplaced)
     (effects (font (size 1.27 1.27)) (justify left))
-    (property "Intersheet References" "${INTERSHEET_REFS}" (id 0) (at 156.0244 89.4556 0)
+    (property "Intersheet References" "${INTERSHEET_REFS}" (id 0) (at 148.4044 89.4556 0)
       (effects (font (size 1.27 1.27)) (justify left) hide)
     )
@@
     )
   )
-  (global_label "GATE" (shape input) (at 200.025 101.6 180) (fields_autoplaced)
+  (global_label "GATE" (shape input) (at 186.055 101.6 180) (fields_autoplaced)
     (effects (font (size 1.27 1.27)) (justify right))
-    (property "Intersheet References" "${INTERSHEET_REFS}" (id 0) (at 193.2256 101.6794 0)
+    (property "Intersheet References" "${INTERSHEET_REFS}" (id 0) (at 179.2556 101.6794 0)
       (effects (font (size 1.27 1.27)) (justify right) hide)
     )
@@
     (pin "1")
   )
-  (symbol (lib_id "Device:R_US") (at 142.24 89.535 90) (mirror x) (unit 1)
+  (symbol (lib_id "Device:R_US") (at 194.31 101.6 90) (mirror x) (unit 1)
     (in_bom yes) (on_board yes)
-    (property "Reference" "R5" (id 0) (at 142.24 92.075 90))
-    (property "Value" "62" (id 1) (at 142.24 87.4546 90))
-    (property "Footprint" "Resistor_SMD:R_0805_2012Metric" (id 2) (at 142.494 90.551 90)
-      (effects (font (size 1.27 1.27)) hide)
-    )
-    (property "Datasheet" "~" (id 3) (at 142.24 89.535 0)
+    (property "Reference" "R5" (id 0) (at 194.31 104.14 90))
+    (property "Value" "10k" (id 1) (at 194.31 99.5196 90))
+    (property "Footprint" "Resistor_SMD:R_0805_2012Metric" (id 2) (at 194.564 102.616 90)
+      (effects (font (size 1.27 1.27)) hide)
+    )
+    (property "Datasheet" "~" (id 3) (at 194.31 101.6 0)
       (effects (font (size 1.27 1.27)) hide)
     )
@@
     )
     (path "/33411cdd-4752-4b5e-9ddb-3f5c464c6578"
-      (reference "R5") (unit 1) (value "62") (footprint "Resistor_SMD:R_0805_2012Metric")
+      (reference "R5") (unit 1) (value "10k") (footprint "Resistor_SMD:R_0805_2012Metric")
     )
     (path "/9812a82a-67c8-4c7e-8eb9-2d5188d40486"
